Commit message: added the movement of the plate

File: urdf_models/panda/panda_arm_balance_bot.urdf (robot description, URDF)
Before this commit: robot panda, 9 links, 8 joints
Links:
- link end-effector: geometry collision cylinder length=0.01 radius=0.2; visual cylinder length=0.012 radius=0.15

Commit message: added the circle in both sense

File: urdf_models/panda/panda_arm_balance_bot.urdf (robot description, URDF)
Before this commit: robot panda, 9 links, 8 joints
Links:
- link end-effector: geometry collision cylinder length=0.01 radius=0.15; visual cylinder length=0.012 radius=0.15

Commit message: Controllers 0 1 2 3 4 implemented

File: urdf_models/panda/panda_arm_balance_bot.urdf (robot description, URDF)
Before this commit: robot panda, 9 links, 8 joints
Links:
- link end-effector: mass 0.2 -> 1.169; geometry collision cylinder length=0.01 radius=0.2; visual cylinder length=0.012 radius=0.2
